File: hardware/amulet.kicad_pcb (KiCad board)
At the start: 2 copper layers, 21 x 21 mm, 31 parts, among them U1 ATtiny84A-MMH, U2 TTP223-BA6, U3 VEML6075

Commit message: Change symbol to pentagram
Parts:
- removed svg2mod: G***, amulet:uvstar1
- added pentagram: G***, amulet:pentagram, F.Cu at (95.9, 95.5)
